File: pcb/makita_aws_rx/makita_aws_rx.kicad_pcb (KiCad board)
At the start: 2 copper layers, 75 x 65 mm, 17 parts, among them J1 MAINS_IN, J2 MAINS_OUT, K2 G5LE-1, Q1 BF244A, SW1 SW_Push

Commit message: PCB nearly done
Parts:
- removed F1: Polyfuse, Capacitor_THT:C_Disc_D5.0mm_W2.5mm_P5.00mm
- added SW3: RESET, Button_Switch_THT:SW_PUSH_6mm_H4.3mm, F.Cu at (166.0, 73.0)
- Q1: value BF244A -> 2N7000
- moved D1 5.69 mm to (198.0, 55.5), turned to 180 degrees
- moved A1 4.88 mm to (188.3, 103.9)
- moved R4 4.77 mm to (205.5, 62.9), turned to -90 degrees
- moved J1 3.04 mm to (194.5, 109.0)
- moved J2 3.04 mm to (211.5, 109.0)
- moved R1 2.92 mm to (195.0, 62.9)
- moved R2 2.92 mm to (198.5, 70.5)
- moved R3 2.92 mm to (202.0, 70.5)
- moved Q1 2.86 mm to (213.5, 58.0)
- moved SW1 1.41 mm to (202.2, 55.5)
Connections:
- A1 pad 1: /SW_PUSH -> /COIL
- A1 pad 2: /LED -> /SW_PUSH
- A1 pad 30: unconnected-(A1-RUN-Pad30) -> /RUN
- A1 pad 4: /COIL -> /LED
- J1 pad 3: Net-(J1-Pin_3) -> /MAINS_L_IN
- Q1 pad 1: Net-(Q1-D) -> GND
- Q1 pad 3: GND -> Net-(Q1-D)
Routing:
- net +5V: track 0.00 -> 120.1 mm
- net /SW_PUSH: track 0.00 -> 65.2 mm
- net Net-(Q1-D): track 0.00 -> 43.0 mm
- net /LED: track 0.00 -> 42.9 mm
- net /MAINS_N: track 0.00 -> 40.8 mm
- net /MAINS_L_IN: track 0.00 -> 40.6 mm
- net /COIL: track 0.00 -> 38.5 mm
- net /MAINS_L_OUT: track 0.00 -> 29.4 mm
- net /MAINS_E: track 0.00 -> 24.9 mm
- net Net-(Q1-G): track 0.00 -> 20.7 mm
- net /RUN: track 0.00 -> 17.6 mm
- net Net-(D1-K): track 0.00 -> 11.7 mm
- net GND: track 0.00 -> 11.2 mm
- added copper zone on B.Cu, net GND
Other:
- board text added: "Makita AWS RX David Turner July 2025"
- board text removed: "Makita AWS RX David Turner - July 2025"

Commit message: Final PCB
Parts:
- J1: value MAINS_IN -> IN
- J2: value MAINS_OUT -> OUT
Connections:
- A1 pad 1: /COIL -> unconnected-(A1-GPIO0-Pad1)
- A1 pad 14: unconnected-(A1-GPIO10-Pad14) -> /COIL
- A1 pad 19: unconnected-(A1-GPIO14-Pad19) -> /SW_PUSH
- A1 pad 2: /SW_PUSH -> unconnected-(A1-GPIO1-Pad2)
- A1 pad 20: unconnected-(A1-GPIO15-Pad20) -> /LED
- A1 pad 4: /LED -> unconnected-(A1-GPIO2-Pad4)
- J1 pad 1: /MAINS_E -> /MAINS_N
- J1 pad 2: /MAINS_N -> /MAINS_E
- J2 pad 1: /MAINS_E -> /MAINS_N
- J2 pad 2: /MAINS_N -> /MAINS_E
Routing:
- net /LED: track 42.9 -> 5.19 mm
- net /SW_PUSH: track 65.2 -> 36.3 mm
- net /COIL: track 38.5 -> 12.0 mm
- net /MAINS_N: track 40.8 -> 48.0 mm
- net /MAINS_L_IN: track 40.6 -> 46.5 mm
- net +5V: track 120.1 -> 124.5 mm
- net Net-(Q1-D): track 43.0 -> 45.4 mm
- net /MAINS_E: track 24.9 -> 26.5 mm
Other:
- board text added: "+"
- board text added: "-"
- board text added: "N E L"
