File: pcb/makita_aws_rx/makita_aws_rx.kicad_sch (KiCad schematic)
At the start: 17 parts, among them J1 MAINS_IN, J2 MAINS_OUT, K2 G5LE-1, Q1 BF244A, SW1 SW_Push

Commit message: PCB nearly done
Parts:
- removed F1: Polyfuse, Capacitor_THT:C_Disc_D5.0mm_W2.5mm_P5.00mm, symbol Device:Polyfuse
- removed Q1: BF244A, Package_TO_SOT_THT:TO-92_Inline, symbol Transistor_FET:BF244A
- added Q1: 2N7000, Package_TO_SOT_THT:TO-92_Inline, symbol Transistor_FET:2N7000
- added SW3: RESET, Button_Switch_THT:SW_PUSH_6mm_H4.3mm, symbol Switch:SW_Push
Connections:
- net COIL: now also A1.1 (GPIO0); no longer A1.4 (GPIO2)
- net GND: now also Q1.1 (S), SW3.1
- net LED: now also A1.4 (GPIO2); no longer A1.2 (GPIO1)
- net MAINS_L_IN: now also J1.3 (Pin_3)
- net SW_PUSH: now also A1.2 (GPIO1); no longer A1.1 (GPIO0)
- net at R2.2, R3.2: now also Q1.2 (G)
- net at K2.2: now also Q1.3 (D)
- net RUN: now reaches A1.30 (RUN)
- net RUN: now also SW3.2
Changed lines of the file:
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@@
+	(wire
+		(pts
+			(xy 246.38 52.07) (xy 246.38 55.88)
+		)
+		(stroke
+			(width 0)
+			(type default)
+		)
+	)
 	(wire
 		(pts
@@
 	(wire
 		(pts
-			(xy 29.21 67.31) (xy 33.02 67.31)
+			(xy 29.21 67.31) (xy 48.26 67.31)
 		)
 		(stroke
@@
 		)
 	)
-	(wire
-		(pts
-			(xy 40.64 67.31) (xy 48.26 67.31)
-		)
-		(stroke
-			(width 0)
-			(type default)
-		)
-	)
 	(label "LED"
-		(at 158.75 66.04 180)
+		(at 158.75 68.58 180)
 		(effects
 			(font
@@
 	)
 	(label "COIL"
-		(at 158.75 68.58 180)
+		(at 158.75 63.5 180)
 		(effects
 			(font
@@
 		)
 	)
+	(label "RUN"
+		(at 158.75 55.88 180)
+		(effects
+			(font
+				(size 1.27 1.27)
+			)
+			(justify right bottom)
+		)
+	)
 	(label "SW_PUSH"
-		(at 158.75 63.5 180)
+		(at 158.75 66.04 180)
+		(effects
+			(font
+				(size 1.27 1.27)
+			)
+			(justify right bottom)
+		)
+	)
+	(label "RUN"
+		(at 246.38 41.91 180)
 		(effects
 			(font
@@
 	)
 	(symbol
+		(lib_id "Transistor_FET:2N7000")
+		(at 123.19 92.71 0)
+		(unit 1)
+		(exclude_from_sim no)
+		(in_bom yes)
+		(on_board yes)
+		(dnp no)
+		(fields_autoplaced yes)
+		(property "Reference" "Q1"
+			(at 129.54 91.4399 0)
+			(effects
+				(font
+					(size 1.27 1.27)
+				)
+				(justify left)
+			)
+		)
+		(property "Value" "2N7000"
+			(at 129.54 93.9799 0)
+			(effects
+				(font
+					(size 1.27 1.27)
+				)
+				(justify left)
+			)
+		)
+		(property "Footprint" "Package_TO_SOT_THT:TO-92_Inline"
+			(at 128.27 94.615 0)
+			(effects
+				(font
+					(size 1.27 1.27)
+					(italic yes)
+				)
+				(justify left)
+				(hide yes)
+			)
+		)
+		(property "Datasheet" "https://www.vishay.com/docs/70226/70226.pdf"
+			(at 128.27 96.52 0)
+			(effects
+				(font
+					(size 1.27 1.27)
+				)
+				(justify left)
+				(hide yes)
+			)
+		)
+		(property "Description" "0.2A Id, 200V Vds, N-Channel MOSFET, 2.6V Logic Level, TO-92"
+			(at 123.19 92.71 0)
+			(effects
+				(font
+					(size 1.27 1.27)
+				)
+				(hide yes)
+			)
+		)
+		(pin "1"
+		)
+		(pin "2"
+		)
+		(pin "3"
+		)
+		(instances
+			(project ""
+				(path "/5e34a7b6-ac3a-4d62-b642-06cd9d5c366e"
+					(reference "Q1")
+					(unit 1)
+				)
+			)
+		)
+	)
+	(symbol
 		(lib_id "power:+5V")
 		(at 86.36 97.79 270)
@@
 	)
 	(symbol
-		(lib_id "Device:Polyfuse")
-		(at 36.83 67.31 90)
-		(unit 1)
-		(exclude_from_sim no)
-		(in_bom yes)
-		(on_board yes)
-		(dnp no)
-		(fields_autoplaced yes)
-		(property "Reference" "F1"
-			(at 36.83 60.96 90)
-			(effects
-				(font
-					(size 1.27 1.27)
-				)
-			)
-		)
-		(property "Value" "Polyfuse"
-			(at 36.83 63.5 90)
-			(effects
-				(font
-					(size 1.27 1.27)
-				)
-			)
-		)
-		(property "Footprint" "Capacitor_THT:C_Disc_D5.0mm_W2.5mm_P5.00mm"
-			(at 41.91 66.04 0)
-			(effects
-				(font
-					(size 1.27 1.27)
-				)
-				(justify left)
-				(hide yes)
-			)
-		)
-		(property "Datasheet" "~"
-			(at 36.83 67.31 0)
-			(effects
-				(font
-					(size 1.27 1.27)
-				)
-				(hide yes)
-			)
-		)
-		(property "Description" "Resettable fuse, polymeric positive temperature coefficient"
-			(at 36.83 67.31 0)
-			(effects
-				(font
-					(size 1.27 1.27)
-				)
-				(hide yes)
-			)
-		)
-		(pin "1"
-		)
-		(pin "2"
-		)
-		(instances
-			(project ""
-				(path "/5e34a7b6-ac3a-4d62-b642-06cd9d5c366e"
-					(reference "F1")
-					(unit 1)
-				)
-			)
-		)
-	)
-	(symbol
 		(lib_id "power:GND")
 		(at 86.36 102.87 90)
@@
 	)
 	(symbol
+		(lib_id "power:GND")
+		(at 246.38 55.88 0)
+		(unit 1)
+		(exclude_from_sim no)
+		(in_bom yes)
+		(on_board yes)
+		(dnp no)
+		(fields_autoplaced yes)
+		(property "Reference" "#PWR012"
+			(at 246.38 62.23 0)
+			(effects
+				(font
+					(size 1.27 1.27)
+				)
+				(hide yes)
+			)
+		)
+		(property "Value" "GND"
+			(at 246.38 60.96 0)
+			(effects
+				(font
+					(size 1.27 1.27)
+				)
+			)
+		)
+		(property "Footprint" ""
+			(at 246.38 55.88 0)
+			(effects
+				(font
+					(size 1.27 1.27)
+				)
+				(hide yes)
+			)
+		)
+		(property "Datasheet" ""
+			(at 246.38 55.88 0)
+			(effects
+				(font
+					(size 1.27 1.27)
+				)
+				(hide yes)
+			)
+		)
+		(property "Description" "Power symbol creates a global label with name \"GND\" , ground"
+			(at 246.38 55.88 0)
+			(effects
+				(font
+					(size 1.27 1.27)
+				)
+				(hide yes)
+			)
+		)
+		(pin "1"
+		)
+		(instances
+			(project ""
+				(path "/5e34a7b6-ac3a-4d62-b642-06cd9d5c366e"
+					(reference "#PWR012")
+					(unit 1)
+				)
+			)
+		)
+	)
+	(symbol
 		(lib_id "Mechanical:MountingHole")
 		(at 25.4 157.48 0)
@@
 	)
 	(symbol
+		(lib_id "Switch:SW_Push")
+		(at 246.38 46.99 90)
+		(unit 1)
+		(exclude_from_sim no)
+		(in_bom yes)
+		(on_board yes)
+		(dnp no)
+		(fields_autoplaced yes)
+		(property "Reference" "SW3"
+			(at 247.65 45.7199 90)
+			(effects
+				(font
+					(size 1.27 1.27)
+				)
+				(justify right)
+			)
+		)
+		(property "Value" "RESET"
+			(at 247.65 48.2599 90)
+			(effects
+				(font
+					(size 1.27 1.27)
+				)
+				(justify right)
+			)
+		)
+		(property "Footprint" "Button_Switch_THT:SW_PUSH_6mm_H4.3mm"
+			(at 241.3 46.99 0)
+			(effects
+				(font
+					(size 1.27 1.27)
+				)
+				(hide yes)
+			)
+		)
+		(property "Datasheet" "~"
+			(at 241.3 46.99 0)
+			(effects
+				(font
+					(size 1.27 1.27)
+				)
+				(hide yes)
+			)
+		)
+		(property "Description" "Push button switch, generic, two pins"
+			(at 246.38 46.99 0)
+			(effects
+				(font
+					(size 1.27 1.27)
+				)
+				(hide yes)
+			)
+		)
+		(pin "1"
+		)
+		(pin "2"
+		)
+		(instances
+			(project "makita_aws_rx"
+				(path "/5e34a7b6-ac3a-4d62-b642-06cd9d5c366e"
+					(reference "SW3")
+					(unit 1)
+				)
+			)
+		)
+	)
+	(symbol
 		(lib_id "Relay:G5LE-1")
 		(at 68.58 74.93 90)
@@
 					(unit 1)
 				)
-			)
-		)
-	)
-	(symbol
-		(lib_id "Transistor_FET:BF244A")
-		(at 123.19 92.71 0)
-		(unit 1)
-		(exclude_from_sim no)
-		(in_bom yes)
-		(on_board yes)
-		(dnp no)
-		(fields_autoplaced yes)
-		(property "Reference" "Q1"
-			(at 128.27 91.4399 0)
-			(effects
-				(font
-					(size 1.27 1.27)
-				)
-				(justify left)
-			)
-		)
-		(property "Value" "BF244A"
-			(at 128.27 93.9799 0)
-			(effects
-				(font
-					(size 1.27 1.27)
-				)
-				(justify left)
-			)
-		)
-		(property "Footprint" "Package_TO_SOT_THT:TO-92_Inline"
-			(at 128.27 94.615 0)
-			(effects
-				(font
-					(size 1.27 1.27)
-					(italic yes)
-				)
-				(justify left)
-				(hide yes)
-			)
-		)
-		(property "Datasheet" "https://media.digikey.com/pdf/Data%20Sheets/Fairchild%20PDFs/BF244x.pdf"
-			(at 128.27 96.52 0)
-			(effects
-				(font
-					(size 1.27 1.27)
-				)
-				(justify left)
-				(hide yes)
-			)
-		)
-		(property "Description" "50mA Id, 30V Vgs, N-Channel FET Transistor, TO-92"
-			(at 123.19 92.71 0)
-			(effects
-				(font
-					(size 1.27 1.27)
-				)
-				(hide yes)
-			)
-		)
-		(pin "3"
-		)
-		(pin "1"
-		)
-		(pin "2"
-		)
-		(instances
-			(project ""
-				(path "/5e34a7b6-ac3a-4d62-b642-06cd9d5c366e"
-					(reference "Q1")
-					(unit 1)
-				)

Commit message: Final PCB
Connections:
- net COIL: now also A1.14 (GPIO10); no longer A1.1 (GPIO0)
- net LED: now also A1.20 (GPIO15); no longer A1.4 (GPIO2)
- net MAINS_E: now also J1.2 (Pin_2), J2.2 (Pin_2); no longer J1.1 (Pin_1), J2.1 (Pin_1)
- net MAINS_N: now also J1.1 (Pin_1), J2.1 (Pin_1); no longer J1.2 (Pin_2), J2.2 (Pin_2)
- net SW_PUSH: now also A1.19 (GPIO14); no longer A1.2 (GPIO1)
- no-connect marks 7 -> 28
Changed lines of the file:
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@@
 	(paper "A4")
 	(junction
-		(at 82.55 97.79)
+		(at 44.45 48.26)
 		(diameter 0)
 		(color 0 0 0 0)
 	)
 	(junction
-		(at 44.45 50.8)
-		(diameter 0)
-		(color 0 0 0 0)
-	)
-	(junction
-		(at 82.55 102.87)
+		(at 53.34 97.79)
 		(diameter 0)
 		(color 0 0 0 0)
@@
 		(color 0 0 0 0)
 	)
+	(junction
+		(at 53.34 102.87)
+		(diameter 0)
+		(color 0 0 0 0)
+	)
+	(no_connect
+		(at 158.75 73.66)
+	)
+	(no_connect
+		(at 158.75 71.12)
+	)
+	(no_connect
+		(at 158.75 83.82)
+	)
+	(no_connect
+		(at 158.75 96.52)
+	)
+	(no_connect
+		(at 158.75 58.42)
+	)
 	(no_connect
 		(at 181.61 40.64)
@@
 	)
 	(no_connect
+		(at 158.75 86.36)
+	)
+	(no_connect
 		(at 204.47 96.52)
 	)
 	(no_connect
+		(at 204.47 76.2)
+	)
+	(no_connect
+		(at 204.47 81.28)
+	)
+	(no_connect
+		(at 204.47 73.66)
+	)
+	(no_connect
+		(at 158.75 66.04)
+	)
+	(no_connect
+		(at 158.75 63.5)
+	)
+	(no_connect
+		(at 204.47 78.74)
+	)
+	(no_connect
+		(at 158.75 81.28)
+	)
+	(no_connect
+		(at 158.75 76.2)
+	)
+	(no_connect
+		(at 158.75 91.44)
+	)
+	(no_connect
+		(at 158.75 68.58)
+	)
+	(no_connect
+		(at 204.47 71.12)
+	)
+	(no_connect
 		(at 204.47 91.44)
 	)
 	(no_connect
+		(at 204.47 68.58)
+	)
+	(no_connect
+		(at 158.75 93.98)
+	)
+	(no_connect
+		(at 204.47 66.04)
+	)
+	(no_connect
 		(at 186.69 40.64)
 	)
@@
 	)
 	(no_connect
+		(at 158.75 78.74)
+	)
+	(no_connect
 		(at 60.96 72.39)
 	)
 	(wire
 		(pts
-			(xy 44.45 50.8) (xy 44.45 102.87)
-		)
-		(stroke
-			(width 0)
-			(type default)
-		)
-	)
-	(wire
-		(pts
 			(xy 125.73 147.32) (xy 125.73 149.86)
 		)
@@
 	(wire
 		(pts
-			(xy 82.55 97.79) (xy 78.74 97.79)
+			(xy 78.74 97.79) (xy 86.36 97.79)
 		)
 		(stroke
@@
 	(wire
 		(pts
-			(xy 25.4 48.26) (xy 93.98 48.26)
+			(xy 25.4 48.26) (xy 44.45 48.26)
 		)
 		(stroke
@@
 	(wire
 		(pts
-			(xy 25.4 50.8) (xy 44.45 50.8)
+			(xy 25.4 50.8) (xy 93.98 50.8)
 		)
 		(stroke
@@
 	(wire
 		(pts
-			(xy 86.36 97.79) (xy 82.55 97.79)
-		)
-		(stroke
-			(width 0)
-			(type default)
-		)
-	)
-	(wire
-		(pts
 			(xy 87.63 135.89) (xy 99.06 135.89)
 		)
@@
 	(wire
 		(pts
+			(xy 53.34 97.79) (xy 58.42 97.79)
+		)
+		(stroke
+			(width 0)
+			(type default)
+		)
+	)
+	(wire
+		(pts
 			(xy 115.57 102.87) (xy 115.57 106.68)
 		)
@@
 	(wire
 		(pts
-			(xy 48.26 97.79) (xy 58.42 97.79)
+			(xy 48.26 97.79) (xy 53.34 97.79)
 		)
 		(stroke
@@
 	(wire
 		(pts
-			(xy 86.36 102.87) (xy 82.55 102.87)
+			(xy 44.45 48.26) (xy 93.98 48.26)
 		)
 		(stroke
@@
 	(wire
 		(pts
-			(xy 44.45 50.8) (xy 93.98 50.8)
-		)
-		(stroke
-			(width 0)
-			(type default)
-		)
-	)
-	(wire
-		(pts
 			(xy 48.26 67.31) (xy 60.96 67.31)
 		)
@@
 	(wire
 		(pts
-			(xy 44.45 102.87) (xy 58.42 102.87)
-		)
-		(stroke
-			(width 0)
-			(type default)
-		)
-	)
-	(wire
-		(pts
-			(xy 82.55 102.87) (xy 78.74 102.87)
+			(xy 44.45 102.87) (xy 53.34 102.87)
+		)
+		(stroke
+			(width 0)
+			(type default)
+		)
+	)
+	(wire
+		(pts
+			(xy 78.74 102.87) (xy 86.36 102.87)
 		)
 		(stroke
@@
 		)
 	)
+	(wire
+		(pts
+			(xy 44.45 48.26) (xy 44.45 102.87)
+		)
+		(stroke
+			(width 0)
+			(type default)
+		)
+	)
+	(wire
+		(pts
+			(xy 53.34 102.87) (xy 58.42 102.87)
+		)
+		(stroke
+			(width 0)
+			(type default)
+		)
+	)
 	(label "LED"
-		(at 158.75 68.58 180)
+		(at 158.75 101.6 180)
 		(effects
 			(font
@@
 	)
 	(label "COIL"
-		(at 158.75 63.5 180)
+		(at 158.75 88.9 180)
 		(effects
 			(font
@@
 	)
 	(label "MAINS_N"
-		(at 58.42 50.8 0)
+		(at 58.42 48.26 0)
 		(effects
 			(font
@@
 	)
 	(label "SW_PUSH"
-		(at 158.75 66.04 180)
+		(at 158.75 99.06 180)
 		(effects
 			(font
@@
 	)
 	(label "MAINS_E"
-		(at 58.42 48.26 0)
+		(at 58.42 50.8 0)
 		(effects
 			(font
@@
 	(symbol
 		(lib_id "power:PWR_FLAG")
-		(at 82.55 102.87 180)
+		(at 53.34 102.87 180)
 		(unit 1)
 		(exclude_from_sim no)
@@
 		(fields_autoplaced yes)
 		(property "Reference" "#FLG02"
-			(at 82.55 104.775 0)
+			(at 53.34 104.775 0)
 			(effects
 				(font
@@
 		)
 		(property "Value" "PWR_FLAG"
-			(at 82.55 107.95 0)
+			(at 53.34 107.95 0)
 			(effects
 				(font
@@
 		)
 		(property "Footprint" ""
-			(at 82.55 102.87 0)
+			(at 53.34 102.87 0)
 			(effects
 				(font
@@
 		)
 		(property "Datasheet" "~"
-			(at 82.55 102.87 0)
+			(at 53.34 102.87 0)
 			(effects
 				(font
@@
 		)
 		(property "Description" "Special symbol for telling ERC where power comes from"
-			(at 82.55 102.87 0)
+			(at 53.34 102.87 0)
 			(effects
 				(font
@@
 	(symbol
 		(lib_id "power:PWR_FLAG")
-		(at 82.55 97.79 0)
+		(at 53.34 97.79 0)
 		(unit 1)
 		(exclude_from_sim no)
@@
 		(fields_autoplaced yes)
 		(property "Reference" "#FLG01"
-			(at 82.55 95.885 0)
+			(at 53.34 95.885 0)
 			(effects
 				(font
@@
 		)
 		(property "Value" "PWR_FLAG"
-			(at 82.55 92.71 0)
+			(at 53.34 92.71 0)
 			(effects
 				(font
@@
 		)
 		(property "Footprint" ""
-			(at 82.55 97.79 0)
+			(at 53.34 97.79 0)
 			(effects
 				(font
@@
 		)
 		(property "Datasheet" "~"
-			(at 82.55 97.79 0)
+			(at 53.34 97.79 0)
 			(effects
 				(font
@@
 		)
 		(property "Description" "Special symbol for telling ERC where power comes from"
-			(at 82.55 97.79 0)
-			(effects
-				(font
+			(at 53.34 97.79 0)
+			(effects
+				(font
